File: KiCad_PCB/KiCad_PCB.kicad_pcb (KiCad board)
At the start: 4 copper layers, 30 x 30 mm, 24 parts, among them J1 530480450, U2 NRF52832-QFAA-R, Y1 ECS-320-8-33B-7KM-TR, Y2 ECS-.327-12.5-12R-TR

Commit message: GBR Files generated
Parts:
- moved R1 5.39 mm to (139.7, 88.9)
Routing:
- net Net-(D1-PadC): track 2.88 -> 3.84 mm
- net GND: vias 25 -> 50
- added copper zone on In1.Cu, net +1V8
- added copper zone on B.Cu, net GND
- added copper zone on F.Cu, net GND
Changed lines of the file:
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@@
   )
   (footprint "Resistor_SMD:R_0603_1608Metric" (layer "F.Cu")
-    (at 138.3 94.1 180)
+    (at 139.7 88.9 180)
     (descr "Resistor SMD 0603 (1608 Metric), square (rectangular) end terminal, IPC_7351 nominal, (Body size source: IPC-SM-782 page 72, https://www.pcb-3d.com/wordpress/wp-content/uploads/ipc-sm-782a_amendment_1_and_2.pdf), generated with kicad-footprint-generator")
     (tags "resistor")
@@
   (segment (start 158.2 102.2) (end 158 102.4) (width 0.25) (layer "B.Cu") (net 1))
   (segment (start 154.578 105.378) (end 154.378 105.578) (width 0.25) (layer "F.Cu") (net 2))
+  (segment (start 156.8 98.5) (end 157.2 98.5) (width 0.5) (layer "F.Cu") (net 2))
   (segment (start 153.378 103.628) (end 153.55 103.8) (width 0.25) (layer "F.Cu") (net 2))
-  (segment (start 156.8 98.5) (end 157.2 98.5) (width 0.5) (layer "F.Cu") (net 2))
+  (segment (start 157.2 98.5) (end 159.1 100.4) (width 0.5) (layer "F.Cu") (net 2))
   (segment (start 157.378 105.378) (end 154.578 105.378) (width 0.25) (layer "F.Cu") (net 2))
   (segment (start 137.6 95.804944) (end 137.474189 95.930755) (width 0.25) (layer "F.Cu") (net 2))
-  (segment (start 157.2 98.5) (end 159.1 100.4) (width 0.5) (layer "F.Cu") (net 2))
   (segment (start 153.378 102.578) (end 153.378 103.628) (width 0.25) (layer "F.Cu") (net 2))
   (segment (start 137.6 95.7) (end 137.6 95.804944) (width 0.25) (layer "F.Cu") (net 2))
   (via (at 153.55 105.7) (size 0.8) (drill 0.4) (layers "F.Cu" "B.Cu") (net 2))
+  (via (at 147.32 85.09) (size 0.8) (drill 0.4) (layers "F.Cu" "B.Cu") (free) (net 2))
+  (via (at 151.13 83.82) (size 0.8) (drill 0.4) (layers "F.Cu" "B.Cu") (free) (net 2))
+  (via (at 158.014538 97.653997) (size 0.8) (drill 0.4) (layers "F.Cu" "B.Cu") (free) (net 2))
   (via (at 152.6 107.6) (size 0.8) (drill 0.4) (layers "F.Cu" "B.Cu") (net 2))
   (via (at 152.6 104.75) (size 0.8) (drill 0.4) (layers "F.Cu" "B.Cu") (net 2))
   (via (at 152.6 103.8) (size 0.8) (drill 0.4) (layers "F.Cu" "B.Cu") (net 2))
   (via (at 155.45 107.6) (size 0.8) (drill 0.4) (layers "F.Cu" "B.Cu") (net 2))
+  (via (at 148.59 83.82) (size 0.8) (drill 0.4) (layers "F.Cu" "B.Cu") (free) (net 2))
   (via (at 153.55 107.6) (size 0.8) (drill 0.4) (layers "F.Cu" "B.Cu") (net 2))
   (via (at 154.5 107.6) (size 0.8) (drill 0.4) (layers "F.Cu" "B.Cu") (net 2))
   (via (at 156.4 106.65) (size 0.8) (drill 0.4) (layers "F.Cu" "B.Cu") (net 2))
   (via (at 153.55 103.8) (size 0.8) (drill 0.4) (layers "F.Cu" "B.Cu") (net 2))
+  (via (at 151.13 85.09) (size 0.8) (drill 0.4) (layers "F.Cu" "B.Cu") (free) (net 2))
   (via (at 156.4 103.8) (size 0.8) (drill 0.4) (layers "F.Cu" "B.Cu") (net 2))
+  (via (at 135.89 101.6) (size 0.8) (drill 0.4) (layers "F.Cu" "B.Cu") (free) (net 2))
   (via (at 154.5 104.75) (size 0.8) (drill 0.4) (layers "F.Cu" "B.Cu") (net 2))
   (via (at 152.6 106.65) (size 0.8) (drill 0.4) (layers "F.Cu" "B.Cu") (net 2))
   (via (at 155.45 105.7) (size 0.8) (drill 0.4) (layers "F.Cu" "B.Cu") (net 2))
+  (via (at 143.51 110.49) (size 0.8) (drill 0.4) (layers "F.Cu" "B.Cu") (free) (net 2))
+  (via (at 148.59 85.09) (size 0.8) (drill 0.4) (layers "F.Cu" "B.Cu") (free) (net 2))
   (via (at 152.6 105.7) (size 0.8) (drill 0.4) (layers "F.Cu" "B.Cu") (net 2))
+  (via (at 149.86 85.09) (size 0.8) (drill 0.4) (layers "F.Cu" "B.Cu") (free) (net 2))
+  (via (at 134.62 96.52) (size 0.8) (drill 0.4) (layers "F.Cu" "B.Cu") (free) (net 2))
   (via (at 154.5 106.65) (size 0.8) (drill 0.4) (layers "F.Cu" "B.Cu") (net 2))
+  (via (at 146.05 85.09) (size 0.8) (drill 0.4) (layers "F.Cu" "B.Cu") (free) (net 2))
+  (via (at 149.86 83.82) (size 0.8) (drill 0.4) (layers "F.Cu" "B.Cu") (free) (net 2))
+  (via (at 155.55652 109.818983) (size 0.8) (drill 0.4) (layers "F.Cu" "B.Cu") (free) (net 2))
+  (via (at 161.736869 101.866793) (size 0.8) (drill 0.4) (layers "F.Cu" "B.Cu") (free) (net 2))
+  (via (at 144.78 83.82) (size 0.8) (drill 0.4) (layers "F.Cu" "B.Cu") (free) (net 2))
   (via (at 153.55 106.65) (size 0.8) (drill 0.4) (layers "F.Cu" "B.Cu") (net 2))
   (via (at 155.45 103.8) (size 0.8) (drill 0.4) (layers "F.Cu" "B.Cu") (net 2))
   (via (at 153.55 104.75) (size 0.8) (drill 0.4) (layers "F.Cu" "B.Cu") (net 2))
   (via (at 154.5 103.8) (size 0.8) (drill 0.4) (layers "F.Cu" "B.Cu") (net 2))
+  (via (at 143.51 83.82) (size 0.8) (drill 0.4) (layers "F.Cu" "B.Cu") (free) (net 2))
   (via (at 154.5 105.7) (size 0.8) (drill 0.4) (layers "F.Cu" "B.Cu") (net 2))
+  (via (at 139.7 105.41) (size 0.8) (drill 0.4) (layers "F.Cu" "B.Cu") (free) (net 2))
+  (via (at 144.78 85.09) (size 0.8) (drill 0.4) (layers "F.Cu" "B.Cu") (free) (net 2))
+  (via (at 140.97 109.22) (size 0.8) (drill 0.4) (layers "F.Cu" "B.Cu") (free) (net 2))
   (via (at 155.45 106.65) (size 0.8) (drill 0.4) (layers "F.Cu" "B.Cu") (net 2))
   (via (at 156.4 105.7) (size 0.8) (drill 0.4) (layers "F.Cu" "B.Cu") (net 2))
+  (via (at 148.197627 100.248255) (size 0.8) (drill 0.4) (layers "F.Cu" "B.Cu") (net 2))
   (via (at 156.4 107.6) (size 0.8) (drill 0.4) (layers "F.Cu" "B.Cu") (net 2))
+  (via (at 143.51 85.09) (size 0.8) (drill 0.4) (layers "F.Cu" "B.Cu") (free) (net 2))
   (via (at 155.45 104.75) (size 0.8) (drill 0.4) (layers "F.Cu" "B.Cu") (net 2))
+  (via (at 147.32 83.82) (size 0.8) (drill 0.4) (layers "F.Cu" "B.Cu") (free) (net 2))
+  (via (at 140.97 100.33) (size 0.8) (drill 0.4) (layers "F.Cu" "B.Cu") (net 2))
+  (via (at 142.24 93.98) (size 0.8) (drill 0.4) (layers "F.Cu" "B.Cu") (net 2))
+  (via (at 146.05 83.82) (size 0.8) (drill 0.4) (layers "F.Cu" "B.Cu") (free) (net 2))
   (via (at 156.4 104.75) (size 0.8) (drill 0.4) (layers "F.Cu" "B.Cu") (net 2))
   (segment (start 156.8 100.4) (end 155.6 99.2) (width 0.25) (layer "F.Cu") (net 3))
@@
   (segment (start 153.4 99) (end 153.4 100.875) (width 0.25) (layer "F.Cu") (net 7))
   (segment (start 152.978 101.422) (end 153.4 101) (width 0.25) (layer "F.Cu") (net 7))
-  (segment (start 136.61 91.8) (end 136.61 93.61) (width 0.25) (layer "F.Cu") (net 8))
-  (segment (start 136.61 93.61) (end 137.1 94.1) (width 0.25) (layer "F.Cu") (net 8))
-  (segment (start 137.1 94.1) (end 137.475 94.1) (width 0.25) (layer "F.Cu") (net 8))
+  (segment (start 136.61 91.165) (end 136.61 91.8) (width 0.25) (layer "F.Cu") (net 8))
+  (segment (start 138.875 88.9) (end 136.61 91.165) (width 0.25) (layer "F.Cu") (net 8))
   (segment (start 157.851946 107.778) (end 159.7 105.929946) (width 0.25) (layer "F.Cu") (net 9))
   (segment (start 159.7 105.929946) (end 159.7 105.6) (width 0.25) (layer "F.Cu") (net 9))
@@
   (segment (start 153.8 93.4) (end 152.2 91.8) (width 0.25) (layer "F.Cu") (net 36))
   (segment (start 153.8 95.2) (end 153.8 93.4) (width 0.25) (layer "F.Cu") (net 36))
+  (segment (start 161 95.475) (end 157.05 91.525) (width 0.25) (layer "F.Cu") (net 42))
   (segment (start 157.05 91.525) (end 157.05 91.1) (width 0.25) (layer "F.Cu") (net 42))
-  (segment (start 161 95.475) (end 157.05 91.525) (width 0.25) (layer "F.Cu") (net 42))
   (segment (start 161 95.475) (end 161 95.4) (width 0.25) (layer "F.Cu") (net 42))
   (segment (start 154.578 96.978) (end 152.65 95.05) (width 0.25) (layer "F.Cu") (net 46))
@@
   (segment (start 150.622 104.178) (end 150 104.8) (width 0.25) (layer "F.Cu") (net 48))
   (segment (start 150 106) (end 149.625 106.375) (width 0.25) (layer "F.Cu") (net 48))
+  (zone (net 2) (net_name "GND") (layer "F.Cu") (hatch edge 0.508)
+    (connect_pads (clearance 0))
+    (min_thickness 0.254) (filled_areas_thickness no)
+    (fill yes (thermal_gap 0.508) (thermal_bridge_width 0.508))
+    (polygon
+      (pts
+        (xy 163.83 113.03)
+        (xy 132.08 113.03)
+        (xy 132.08 81.28)
+        (xy 163.83 81.28)
+      )
+    )
+  )
+  (zone (net 0) (net_name "") (layers "F.Cu" "In1.Cu" "In2.Cu" "B.Cu") (hatch edge 0.508)
+    (connect_pads (clearance 0))
+    (min_thickness 0.254)
+    (keepout (tracks not_allowed) (vias not_allowed) (pads not_allowed ) (copperpour not_allowed) (footprints allowed))
+    (fill (thermal_gap 0.508) (thermal_bridge_width 0.508))
+    (polygon
+      (pts
+        (xy 162.56 86.36)
+        (xy 162.56 93.98)
+        (xy 157.48 93.98)
+        (xy 153.67 91.44)
+        (xy 153.67 82.55)
+        (xy 160.02 82.55)
+      )
+    )
+  )
+  (zone (net 1) (net_name "+1V8") (layer "In1.Cu") (hatch edge 0.508)
+    (connect_pads (clearance 0))
+    (min_thickness 0.254) (filled_areas_thickness no)
+    (fill yes (thermal_gap 0.508) (thermal_bridge_width 0.508))
+    (polygon
+      (pts
+        (xy 163.83 113.03)
+        (xy 132.08 113.03)
+        (xy 132.08 81.28)
+        (xy 163.83 81.28)
+      )
+    )
+  )
+  (zone (net 2) (net_name "GND") (layer "B.Cu") (hatch edge 0.508)
+    (connect_pads (clearance 0))
+    (min_thickness 0.254) (filled_areas_thickness no)
+    (fill yes (thermal_gap 0.508) (thermal_bridge_width 0.508))
+    (polygon
+      (pts
+        (xy 163.83 113.03)
+        (xy 132.08 113.03)
+        (xy 132.08 81.28)
+        (xy 163.83 81.28)
+      )
+    )
+  )
 )
